File: cad_files/SERVOx16.kicad_pcb (KiCad board)
At the start: 2 copper layers, 49 x 85 mm, 57 parts, among them J1 USB_C_Receptacle_USB2.0, J10 Conn_01x08, J11 Conn_01x08, J12 Conn_01x08, J13 Conn_01x08, J2 RJ11, J3 RJ11, J4 PH, J5 PH, J6 Conn_02x03_Odd_Even, J7 Conn_01x02, J8 Conn_01x08, J9 Conn_01x08, SW1 SW_Push, SW2 SW_Push, SW3 SW_Push, U1 SY8401ABC, U2 AMS1117-3.3, U3 EDGE_STM32F405_CPU_V1, U5 PCA9685PW, U6 SWITCH_5-WAY_TACTIL_10X10

Commit message: update documentation
Parts:
- removed H1: MountingHole, Evezor_extras:OLED_STANDOFF
- J6: footprint Evezor_extras:OLED_HEADER -> Connector_PinSocket_2.54mm:PinSocket_2x03_P2.54mm_Vertical_SMD
Connections:
- SW2 pad 1: /BUTTON_A -> /BUTTON_B
- SW3 pad 1: /BUTTON_B -> /BUTTON_A
- U3 pad 15: /BUTTON_B -> /BUTTON_A
- U3 pad 16: /BUTTON_A -> /BUTTON_B
Routing:
- net /BUTTON_B: track 6.91 -> 15.6 mm
- net /BUTTON_A: track 15.6 -> 6.91 mm
Changed lines of the file:
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@@
     (tracks 840)
     (zones 0)
-    (modules 57)
+    (modules 56)
     (nets 90)
   )
@@
     (47 F.CrtYd user)
     (48 B.Fab user hide)
-    (49 F.Fab user hide)
+    (49 F.Fab user)
   )
   (setup
@@
     (add_net VBUS)
   )
-  (module Evezor_extras:OLED_HEADER (layer F.Cu)
+  (module Connector_PinSocket_2.54mm:PinSocket_2x03_P2.54mm_Vertical_SMD (layer F.Cu)
     (at 105 104.5)
     (descr "surface-mounted straight socket strip, 2x03, 2.54mm pitch, double cols (from Kicad 4.0.7), script generated")
     (tags "Surface mounted socket strip SMD 2x03 2.54mm double row")
     (attr smd)
-    (fp_text reference J6 (at 0 -5.31) (layer F.Fab)
+    (fp_text reference J6 (at 0 -5.31) (layer F.SilkS)
       (effects (font (size 1 1) (thickness 0.15)))
     )
@@
       (rotate (xyz 0 0 0))
     )
-    (model ${EVEZOR}/oled_shield.step
-      (offset (xyz 21.25 1.5 11.5))
-      (scale (xyz 1 1 1))
-      (rotate (xyz 0 0 0))
-    )
-  )
-  (module Evezor_extras:OLED_STANDOFF (layer F.Cu)
-    (at 145 104)
-    (fp_text reference H1 (at -0.0635 3.302) (layer F.SilkS)
-      (effects (font (size 1 1) (thickness 0.15)))
-    )
-    (fp_text value MountingHole (at -0.0635 -5.461) (layer F.Fab)
-      (effects (font (size 1 1) (thickness 0.15)))
-    )
-    (pad "" np_thru_hole circle (at 0 0) (size 3.1 3.1) (drill 3.1) (layers *.Cu *.Mask))
-    (model "${EVEZOR}/M3 STANDOFF_lcd.step"
-      (offset (xyz 0 0 -0.15))
-      (scale (xyz 1 1 1))
-      (rotate (xyz 0 0 0))
-    )
   )
   (module Evezor_BUTTONS:SWITCH_5WAY_10x10 (layer F.Cu)
@@
       (net 4 GND))
     (pad 1 smd rect (at -3.85 0) (size 1.5 1.2) (layers F.Cu F.Paste F.Mask)
-      (net 77 /BUTTON_B))
+      (net 76 /BUTTON_A))
     (model "${EVEZOR}/Green Tactile Switch - Green Tactile Switch.step"
       (at (xyz 0 0 0))
@@
       (net 4 GND))
     (pad 1 smd rect (at -3.85 0) (size 1.5 1.2) (layers F.Cu F.Paste F.Mask)
-      (net 76 /BUTTON_A))
+      (net 77 /BUTTON_B))
     (model "${EVEZOR}/Green Tactile Switch - Green Tactile Switch.step"
       (at (xyz 0 0 0))
@@
       (net 14 "Net-(U3-Pad14)") (zone_connect 1) (thermal_width 0.5))
     (pad 15 smd rect (at -10.9 5.3 90) (size 0.9 2) (layers B.Cu B.Paste B.Mask)
-      (net 77 /BUTTON_B) (zone_connect 1) (thermal_width 0.5))
+      (net 76 /BUTTON_A) (zone_connect 1) (thermal_width 0.5))
     (pad 28 smd rect (at 10.9 4 90) (size 0.9 2) (layers B.Cu B.Paste B.Mask)
       (net 13 "Net-(U3-Pad28)") (zone_connect 1) (thermal_width 0.5))
     (pad 16 smd rect (at -10.9 4 90) (size 0.9 2) (layers B.Cu B.Paste B.Mask)
-      (net 76 /BUTTON_A) (zone_connect 1) (thermal_width 0.5))
+      (net 77 /BUTTON_B) (zone_connect 1) (thermal_width 0.5))
     (pad 27 smd rect (at 6.5 -0.4) (size 0.9 2) (layers B.Cu B.Paste B.Mask)
       (net 6 /CAN_L) (zone_connect 1) (thermal_width 0.5))
@@
   (segment (start 143.81 74) (end 143.81 70.91) (width 2) (layer F.Cu) (net 75))
   (segment (start 143.81 70.91) (end 142.1 69.2) (width 2) (layer F.Cu) (net 75))
-  (via (at 132.01 117.27) (size 0.8) (drill 0.4) (layers F.Cu B.Cu) (net 76))
-  (segment (start 134.34 119.6) (end 132.409999 117.669999) (width 0.3) (layer B.Cu) (net 76))
-  (segment (start 135.84 119.6) (end 134.34 119.6) (width 0.3) (layer B.Cu) (net 76))
-  (segment (start 132.409999 117.669999) (end 132.01 117.27) (width 0.3) (layer B.Cu) (net 76))
-  (segment (start 131.444315 117.27) (end 132.01 117.27) (width 0.3) (layer F.Cu) (net 76))
-  (segment (start 129.15 109.9) (end 128.97 110.08) (width 0.3) (layer F.Cu) (net 76))
-  (segment (start 128.97 110.08) (end 128.97 115.97) (width 0.3) (layer F.Cu) (net 76))
-  (segment (start 130.2 109.9) (end 129.15 109.9) (width 0.3) (layer F.Cu) (net 76))
-  (segment (start 130.27 117.27) (end 131.444315 117.27) (width 0.3) (layer F.Cu) (net 76))
-  (segment (start 128.97 115.97) (end 130.27 117.27) (width 0.3) (layer F.Cu) (net 76))
-  (via (at 133.33 117.2) (size 0.8) (drill 0.4) (layers F.Cu B.Cu) (net 77))
-  (segment (start 135.84 118.3) (end 134.43 118.3) (width 0.3) (layer B.Cu) (net 77))
-  (segment (start 134.43 118.3) (end 133.33 117.2) (width 0.3) (layer B.Cu) (net 77))
-  (segment (start 131.13 115) (end 130.3 115) (width 0.3) (layer F.Cu) (net 77))
-  (segment (start 133.33 117.2) (end 131.13 115) (width 0.3) (layer F.Cu) (net 77))
+  (via (at 132.01 117.27) (size 0.8) (drill 0.4) (layers F.Cu B.Cu) (net 77))
+  (segment (start 134.34 119.6) (end 132.409999 117.669999) (width 0.3) (layer B.Cu) (net 77))
+  (segment (start 135.84 119.6) (end 134.34 119.6) (width 0.3) (layer B.Cu) (net 77))
+  (segment (start 132.409999 117.669999) (end 132.01 117.27) (width 0.3) (layer B.Cu) (net 77))
+  (segment (start 131.444315 117.27) (end 132.01 117.27) (width 0.3) (layer F.Cu) (net 77))
+  (segment (start 129.15 109.9) (end 128.97 110.08) (width 0.3) (layer F.Cu) (net 77))
+  (segment (start 128.97 110.08) (end 128.97 115.97) (width 0.3) (layer F.Cu) (net 77))
+  (segment (start 130.2 109.9) (end 129.15 109.9) (width 0.3) (layer F.Cu) (net 77))
+  (segment (start 130.27 117.27) (end 131.444315 117.27) (width 0.3) (layer F.Cu) (net 77))
+  (segment (start 128.97 115.97) (end 130.27 117.27) (width 0.3) (layer F.Cu) (net 77))
+  (via (at 133.33 117.2) (size 0.8) (drill 0.4) (layers F.Cu B.Cu) (net 76))
+  (segment (start 135.84 118.3) (end 134.43 118.3) (width 0.3) (layer B.Cu) (net 76))
+  (segment (start 134.43 118.3) (end 133.33 117.2) (width 0.3) (layer B.Cu) (net 76))
+  (segment (start 131.13 115) (end 130.3 115) (width 0.3) (layer F.Cu) (net 76))
+  (segment (start 133.33 117.2) (end 131.13 115) (width 0.3) (layer F.Cu) (net 76))
   (segment (start 114.04 117) (end 116.63 117) (width 0.3) (layer B.Cu) (net 78))
   (segment (start 116.63 117) (end 117.77 118.14) (width 0.3) (layer B.Cu) (net 78))
